Commit message: feat: Update motoman_mh5_support/urdf/mh5_2f85.xacro
This commit updates the motoman_mh5_support/urdf/mh5_2f85.xacro file. Changes include adding parameters for use_fake_hardware and parent, importing macros, and modifying the robotiq_gripper element. These updates improve the configurability and functionality of the MH5 robot's URDF file.

File: motoman_mh5_support/urdf/mh5_2f85.urdf (robot description, URDF)
Before this commit: robot motoman_mh5_2f85, 16 links, 15 joints
Links:
- link robotiq_85_base_link: geometry collision mesh filename=file:///motoman/install/robotiq_description/share/robotiq_d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; visual mesh filename=file:///motoman/install/robotiq_description/share/robotiq_d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
- link robotiq_85_left_finger_link: geometry collision mesh filename=file:///motoman/install/robotiq_description/share/robotiq_d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; visual mesh filename=file:///motoman/install/robotiq_description/share/robotiq_d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
- link robotiq_85_left_finger_tip_link: geometry collision mesh filename=file:///motoman/install/robotiq_description/share/robotiq_d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; visual mesh filename=file:///motoman/install/robotiq_description/share/robotiq_d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
- link robotiq_85_left_inner_knuckle_link: geometry collision mesh filename=file:///motoman/install/robotiq_description/share/robotiq_d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; visual mesh filename=file:///motoman/install/robotiq_description/share/robotiq_d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
- link robotiq_85_left_knuckle_link: geometry collision mesh filename=file:///motoman/install/robotiq_description/share/robotiq_d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; visual mesh filename=file:///motoman/install/robotiq_description/share/robotiq_d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
- link robotiq_85_right_finger_link: geometry collision mesh filename=file:///motoman/install/robotiq_description/share/robotiq_d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; visual mesh filename=file:///motoman/install/robotiq_description/share/robotiq_d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
- link robotiq_85_right_finger_tip_link: geometry collision mesh filename=file:///motoman/install/robotiq_description/share/robotiq_d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; visual mesh filename=file:///motoman/install/robotiq_description/share/robotiq_d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
- link robotiq_85_right_inner_knuckle_link: geometry collision mesh filename=file:///motoman/install/robotiq_description/share/robotiq_d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; visual mesh filename=file:///motoman/install/robotiq_description/share/robotiq_d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
- link robotiq_85_right_knuckle_link: geometry collision mesh filename=file:///motoman/install/robotiq_description/share/robotiq_d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; visual mesh filename=file:///motoman/install/robotiq_description/share/robotiq_d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

File: motoman_mh5_support/urdf/mh5_2f85.xacro (robot description, xacro)
@@ -1,8 +1,13 @@
 <?xml version="1.0" ?>
 <robot name="motoman_mh5_2f85" xmlns:xacro="http://ros.org/wiki/xacro">
+    <!-- parameters -->
+    <xacro:arg name="use_fake_hardware" default="true" />
+    <xacro:arg name="parent" default="link_t" />
+    <!-- Import macros -->
     <xacro:include filename="$(find motoman_mh5_support)/urdf/mh5_macro.xacro" />
     <xacro:include filename="$(find robotiq_description)/urdf/robotiq_2f_85_macro.urdf.xacro" />
     <xacro:motoman_mh5 prefix=""/>
-    <xacro:robotiq_gripper name="robotiq_2f85" prefix="" parent="link_t">
+    <!-- <xacro:robotiq_gripper name="robotiq_2f85" prefix="" parent="link_t"> -->
+    <xacro:robotiq_gripper name="RobotiqGripperHardwareInterface" prefix="" parent="$(arg parent)" use_fake_hardware="$(arg use_fake_hardware)">
         <origin xyz="0 0 0" rpy="1.5708 0 1.5708" />
     </xacro:robotiq_gripper>
