Commit message: feat: Refect urdf and control of motoman_mh5

File: motoman_mh5_moveit_config/config/motoman_mh5.ros2_control.xacro (robot description, xacro)
@@ -1,10 +1,17 @@
 <?xml version="1.0"?>
 <robot xmlns:xacro="http://www.ros.org/wiki/xacro">
-    <xacro:macro name="motoman_mh5_ros2_control" params="name initial_positions_file">
+    <xacro:macro name="motoman_mh5_ros2_control" params="name initial_positions_file use_fake_hardware">
         <xacro:property name="initial_positions" value="${load_yaml(initial_positions_file)['initial_positions']}"/>
+        <xacro:property name="fake_hardware" value="${use_fake_hardware}"/>
         <ros2_control name="${name}" type="system">
             <hardware>
-                <!-- By default, set up controllers for simulation. This won't work on real hardware -->
-                <plugin>mock_components/GenericSystem</plugin>
+                <xacro:if value="${fake_hardware}">
+                  <!-- By default, set up controllers for simulation. This won't work on real hardware -->
+                  <plugin>mock_components/GenericSystem</plugin>
+                </xacro:if>
+                <xacro:unless value="${fake_hardware}">
+                  <!-- By default, set up controllers for simulation. This won't work on real hardware -->
+                  <plugin>mock_components/GenericSystem</plugin>
+                </xacro:unless>
             </hardware>
             <joint name="joint_s">
@@ -13,5 +20,5 @@
                   <param name="initial_value">${initial_positions['joint_s']}</param>
                 </state_interface>
-                <state_interface name="velocity"/>
+                <!-- <state_interface name="velocity"/> -->
             </joint>
             <joint name="joint_l">
@@ -20,5 +27,5 @@
                   <param name="initial_value">${initial_positions['joint_l']}</param>
                 </state_interface>
-                <state_interface name="velocity"/>
+                <!-- <state_interface name="velocity"/> -->
             </joint>
             <joint name="joint_u">
@@ -27,5 +34,5 @@
                   <param name="initial_value">${initial_positions['joint_u']}</param>
                 </state_interface>
-                <state_interface name="velocity"/>
+                <!-- <state_interface name="velocity"/> -->
             </joint>
             <joint name="joint_r">
@@ -34,5 +41,5 @@
                   <param name="initial_value">${initial_positions['joint_r']}</param>
                 </state_interface>
-                <state_interface name="velocity"/>
+                <!-- <state_interface name="velocity"/> -->
             </joint>
             <joint name="joint_b">
@@ -41,5 +48,5 @@
                   <param name="initial_value">${initial_positions['joint_b']}</param>
                 </state_interface>
-                <state_interface name="velocity"/>
+                <!-- <state_interface name="velocity"/> -->
             </joint>
             <joint name="joint_t">
@@ -48,5 +55,5 @@
                   <param name="initial_value">${initial_positions['joint_t']}</param>
                 </state_interface>
-                <state_interface name="velocity"/>
+                <!-- <state_interface name="velocity"/> -->
             </joint>
         </ros2_control>

File: motoman_mh5_moveit_config/config/motoman_mh5.urdf.xacro (robot description, xacro)
@@ -1,9 +1,25 @@
 <?xml version="1.0"?>
 <robot xmlns:xacro="http://www.ros.org/wiki/xacro" name="motoman_mh5">
+    <!-- Arguments -->
     <xacro:arg name="initial_positions_file" default="initial_positions.yaml" />
+    <xacro:arg name="use_fake_hardware" default="true"/>
+    <xacro:arg name="attach_2f85" default="true"/>
+    <xacro:arg name="parent" default="link_t"/>
+    <xacro:arg name="prefix" default=""/>
     <!-- Import motoman_mh5 urdf file -->
-    <xacro:include filename="$(find motoman_mh5_support)/urdf/mh5.urdf" />
+    <xacro:include filename="$(find motoman_mh5_support)/urdf/mh5_macro.xacro" />
+    <xacro:include filename="$(find robotiq_description)/urdf/robotiq_2f_85_macro.urdf.xacro" />
     <!-- Import control_xacro -->
     <xacro:include filename="motoman_mh5.ros2_control.xacro" />
-    <xacro:motoman_mh5_ros2_control name="FakeSystem" initial_positions_file="$(arg initial_positions_file)"/>
+    <xacro:if value="$(arg use_fake_hardware)">
+        <xacro:motoman_mh5_ros2_control name="MH5System" initial_positions_file="$(arg initial_positions_file)" use_fake_hardware="$(arg use_fake_hardware)"/>
+    </xacro:if>
+    <!-- Motoman MH5 -->
+	<xacro:motoman_mh5 prefix="$(arg prefix)"/>
+    <!-- Robotiq 2F85 -->
+    <xacro:if value="$(arg attach_2f85)">
+        <xacro:robotiq_gripper name="RobotiqGripperHardwareInterface" prefix="$(arg prefix)" parent="$(arg parent)" use_fake_hardware="$(arg use_fake_hardware)">
+            <origin xyz="0 0 0" rpy="1.5708 0 1.5708" />
+        </xacro:robotiq_gripper>
+    </xacro:if>
 </robot>
