Commit message: Add GP25-12 model to motoman_gp25_support (#608)
Squashed commits:

* Add GP25-12 model to motoman_gp25_support
   Added the Yaskawa Motoman GP25-12 robot model to the motoman_gp25_support as a variant.
   Updated the GP25 model and made small corrections.
* Avoid dashes in filenames
* Update references to GP-25 resources
* Always provide joint names config
* Formatting
* Formatting: trailing whitespace, more tabs-to-spaces
* Update motoman_gp25_support/launch/test_gp25_12.launch
* Clarify status of OPW parameters

---------

Co-authored-by: gavanderhoorn <g.a.vanderhoorn@tudelft.nl>

File: motoman_gp25_support/urdf/gp25.xacro (robot description, xacro)
@@ -1,5 +1,5 @@
 <?xml version="1.0" ?>
 <robot name="motoman_gp25" xmlns:xacro="http://ros.org/wiki/xacro">
-	<xacro:include filename="$(find motoman_gp25_support)/urdf/gp25_macro.xacro" />
-	<xacro:motoman_gp25 prefix=""/>
+  <xacro:include filename="$(find motoman_gp25_support)/urdf/gp25_macro.xacro" />
+  <xacro:motoman_gp25 prefix=""/>
 </robot>

File: motoman_gp25_support/urdf/gp25_12_macro.xacro (robot description, xacro)
@@ -1,5 +1,5 @@
 <?xml version="1.0" ?>
 <robot xmlns:xacro="http://ros.org/wiki/xacro">
-<xacro:macro name="motoman_gp25" params="prefix">
+<xacro:macro name="motoman_gp25_12" params="prefix">
     <xacro:include filename="$(find motoman_resources)/urdf/common_materials.xacro"/>
     <!-- link list -->
@@ -59,5 +59,5 @@
         <visual>
             <geometry>
-                <mesh filename="package://motoman_gp25_support/meshes/gp25/visual/link_4_r.dae"/>
+                <mesh filename="package://motoman_gp25_support/meshes/gp25_12/visual/link_4_r.dae"/>
             </geometry>
             <xacro:material_yaskawa_blue/>
@@ -65,5 +65,5 @@
         <collision>
             <geometry>
-                <mesh filename="package://motoman_gp25_support/meshes/gp25/collision/link_4_r.stl"/>
+                <mesh filename="package://motoman_gp25_support/meshes/gp25_12/collision/link_4_r.stl"/>
             </geometry>
         </collision>
@@ -116,12 +116,12 @@
         <origin xyz="0 0 0.760" rpy="0 0 0" />
         <axis xyz="0 -1 0" />
-        <limit lower="${radians(-86)}" upper="${radians(160)}" effort="926.1" velocity="${radians(265)}"/>
+        <limit lower="${radians(-86)}" upper="${radians(160)}" effort="926.1" velocity="${radians(220)}"/>
     </joint>
     <joint name="${prefix}joint_4_r" type="revolute">
         <parent link="${prefix}link_3_u"/>
         <child link="${prefix}link_4_r"/>
-        <origin xyz="0.795 0 0.200" rpy="0 0 0" />
+        <origin xyz="1.082 0 0.200" rpy="0 0 0" />
         <axis xyz="-1 0 0" />
-        <limit lower="${radians(-200)}" upper="${radians(200)}" effort="88.2" velocity="${radians(420)}"/>
+        <limit lower="${radians(-200)}" upper="${radians(200)}" effort="78.4" velocity="${radians(435)}"/>
     </joint>
     <joint name="${prefix}joint_5_b" type="revolute">
@@ -130,5 +130,5 @@
         <origin xyz="0 0 0" rpy="0 0 0" />
         <axis xyz="0 -1 0" />
-        <limit lower="${radians(-150)}" upper="${radians(150)}" effort="70.56" velocity="${radians(420)}"/>
+        <limit lower="${radians(-150)}" upper="${radians(150)}" effort="67.0" velocity="${radians(435)}"/>
     </joint>
     <joint name="${prefix}joint_6_t" type="revolute">
@@ -137,5 +137,5 @@
         <origin xyz="0 0 0" rpy="0 0 0" />
         <axis xyz="-1 0 0" />
-        <limit lower="${radians(-455)}" upper="${radians(455)}" effort="50.31" velocity="${radians(885)}"/>
+        <limit lower="${radians(-455)}" upper="${radians(455)}" effort="33.3" velocity="${radians(700)}"/>
     </joint>
     <!-- end of joint list -->
