Commit message: Use radians(..) with limits from HW1486547
Easier to compare/check.

File: motoman_gp7_support/urdf/gp7_macro.xacro (robot description, xacro)
@@ -102,5 +102,5 @@
         <origin xyz="0 0 0.330" rpy="0 0 0" />
         <axis xyz="0 0 1" />
-        <limit lower="-2.9670" upper="2.9670" effort="212.66" velocity="6.5449"/>
+        <limit lower="${radians(-170)}" upper="${radians(170)}" effort="212.66" velocity="${radians(375)}"/>
     </joint>
     <joint name="${prefix}joint_2_l" type="revolute">
@@ -109,5 +109,5 @@
         <origin xyz="0.040 0 0" rpy="0 0 0" />
         <axis xyz="0 1 0" />
-        <limit lower="-1.1344" upper="2.5307" effort="205.80" velocity="5.4977"/>
+        <limit lower="${radians(-65)}" upper="${radians(145)}" effort="205.80" velocity="${radians(315)}"/>
     </joint>
     <joint name="${prefix}joint_3_u" type="revolute">
@@ -116,5 +116,5 @@
         <origin xyz="0 0 0.445" rpy="0 0 0" />
         <axis xyz="0 -1 0" />
-        <limit lower="-1.2217" upper="3.3161" effort="106.82" velocity="7.1558"/>
+        <limit lower="${radians(-70)}" upper="${radians(190)}" effort="106.82" velocity="${radians(410)}"/>
     </joint>
     <joint name="${prefix}joint_4_r" type="revolute">
@@ -123,5 +123,5 @@
         <origin xyz="0.440 0 0.040" rpy="0 0 0" />
         <axis xyz="-1 0 0" />
-        <limit lower="-3.3161" upper="3.3161" effort="55.86" velocity="9.5993"/>
+        <limit lower="${radians(-190)}" upper="${radians(190)}" effort="55.86" velocity="${radians(550)}"/>
     </joint>
     <joint name="${prefix}joint_5_b" type="revolute">
@@ -130,5 +130,5 @@
         <origin xyz="0 0 0" rpy="0 0 0" />
         <axis xyz="0 -1 0" />
-        <limit lower="-2.3561" upper="2.3561" effort="32.68" velocity="9.5993"/>
+        <limit lower="${radians(-135)}" upper="${radians(135)}" effort="32.68" velocity="${radians(550)}"/>
     </joint>
     <joint name="${prefix}joint_6_t" type="revolute">
@@ -137,5 +137,5 @@
         <origin xyz="0 0 0" rpy="0 0 0" />
         <axis xyz="-1 0 0" />
-        <limit lower="-6.2831" upper="6.2831" effort="22.54" velocity="17.4533"/>
+        <limit lower="${radians(-360)}" upper="${radians(360)}" effort="22.54" velocity="${radians(1000)}"/>
     </joint>
     <!-- end of joint list -->
