Commit message: Tabs -> spaces

File: motoman_hc20_support/urdf/hc30pl_macro.xacro (robot description, xacro)
@@ -74,5 +74,5 @@
           <mesh filename="package://motoman_hc20_support/meshes/hc20dtp/visual/link_5_b.dae"/>
         </geometry>
-		<origin rpy="0 1.57075 0"/>
+        <origin rpy="0 1.57075 0"/>
         <xacro:material_yaskawa_white/>
       </visual>
@@ -81,5 +81,5 @@
           <mesh filename="package://motoman_hc20_support/meshes/hc20dtp/collision/link_5_b.stl"/>
         </geometry>
-		<origin rpy="0 1.57075 0"/>
+        <origin rpy="0 1.57075 0"/>
       </collision>
     </link>
@@ -89,5 +89,5 @@
           <mesh filename="package://motoman_hc20_support/meshes/hc20dtp/visual/link_6_t.dae"/>
         </geometry>
-		<origin rpy="0 1.57075 0"/>
+        <origin rpy="0 1.57075 0"/>
         <xacro:material_yaskawa_white/>
       </visual>
@@ -96,5 +96,5 @@
           <mesh filename="package://motoman_hc20_support/meshes/hc20dtp/collision/link_6_t.stl"/>
         </geometry>
-		<origin rpy="0 1.57075 0"/>
+        <origin rpy="0 1.57075 0"/>
       </collision>
     </link>

Commit message: Updated package description about HC30PL limitation
Added note about HC30PL limitation about the flange needing to point downward which cannot be accounted for by the URDF file. Increase B-axis motion so that compounded angles of the L,U and B axes can keep the flange model with 15 degrees of the ground.
Reverted package version to 0.1.0

File: motoman_hc20_support/urdf/hc30pl_macro.xacro (robot description, xacro)
@@ -134,5 +134,5 @@
       <origin xyz="0 0 0" rpy="0 0 0" />
       <axis xyz="0 -1 0" />
-      <limit lower="${radians(-15)}" upper="${radians(15)}" effort="141.12" velocity="${radians(132)}"/>
+      <limit lower="${radians(-180)}" upper="${radians(180)}" effort="141.12" velocity="${radians(132)}"/>
     </joint>
     <joint name="${prefix}joint_6_t" type="revolute">

Commit message: Update HC30PL motion and speed limits
Correct on the HC30PL motion and speed range (R and B axes)

File: motoman_hc20_support/urdf/hc30pl_macro.xacro (robot description, xacro)
@@ -113,5 +113,5 @@
       <origin xyz="0 0 0" rpy="0 0 0" />
       <axis xyz="0 1 0" />
-      <limit lower="${radians(-154)}" upper="${radians(180)}" effort="1223.04" velocity="${radians(80)}"/>
+      <limit lower="${radians(-180)}" upper="${radians(180)}" effort="1223.04" velocity="${radians(80)}"/>
     </joint>
     <joint name="${prefix}joint_3_u" type="revolute">
@@ -127,5 +127,5 @@
       <origin xyz="0.880 0 0" rpy="0 0 0" />
       <axis xyz="-1 0 0" />
-      <limit lower="${radians(-15)}" upper="${radians(15)}" effort="368.48" velocity="${radians(112)}"/>
+      <limit lower="${radians(-210)}" upper="${radians(210)}" effort="368.48" velocity="${radians(130)}"/>
     </joint>
     <joint name="${prefix}joint_5_b" type="revolute">
@@ -134,5 +134,5 @@
       <origin xyz="0 0 0" rpy="0 0 0" />
       <axis xyz="0 -1 0" />
-      <limit lower="${radians(-180)}" upper="${radians(180)}" effort="141.12" velocity="${radians(132)}"/>
+      <limit lower="${radians(-90)}" upper="${radians(270)}" effort="141.12" velocity="${radians(180)}"/>
     </joint>
     <joint name="${prefix}joint_6_t" type="revolute">
