Commit message: Correct velocity limit
and add manual information & reference.

File: motoman_motopos_mh1655_support/urdf/motopos_mh1655_macro.xacro (robot description, xacro)
@@ -53,5 +53,7 @@
       <origin xyz="0 0 0.305" rpy="0 0 0"/>
       <axis xyz="1 0 0"/>
-      <limit lower="${-2*pi}" upper="${2*pi}" effort="1274" velocity="1.3962"/>
+      <!-- NOTE: the velocity limit is a conservative conversion from the stated
+           limit in the manual: 10.8 rpm (in section 3.2.1) -->
+      <limit lower="${-2*pi}" upper="${2*pi}" effort="1274" velocity="1.1309"/>
     </joint>
     <!-- end of joint list -->
