Commit message: mh12: state documentation used
And make sure joint limits correspond to what that documentation specs
(by switching to the `radians(..)` helper function instead of manually
converted limits in rad and rad/s).

File: motoman_mh12_support/urdf/mh12_macro.xacro (robot description, xacro)
@@ -103,5 +103,5 @@
         <origin xyz="0 0 0.450" rpy="0 0 0" />
         <axis xyz="0 0 1" />
-    <limit  lower="-2.9670" upper="2.9670" effort="648.27" velocity="3.8397" />
+        <limit lower="${radians(-170)}" upper="${radians(170)}" effort="648.27" velocity="${radians(220)}" />
     </joint>
     <joint name="${prefix}joint_2_l" type="revolute">
@@ -110,5 +110,5 @@
         <origin xyz="0.155 0 0" rpy="0 0 0" />
         <axis xyz="0 1 0" />
-        <limit lower="-1.5708" upper="2.7052" effort="874.65" velocity="3.4906"/>
+        <limit lower="${radians(-90)}" upper="${radians(155)}" effort="874.65" velocity="${radians(200)}"/>
     </joint>
     <joint name="${prefix}joint_3_u" type="revolute">
@@ -117,5 +117,5 @@
         <origin xyz="0 0 0.614" rpy="0 0 0" />
         <axis xyz="0 -1 0" />
-        <limit lower="-1.4835" upper="2.6179" effort="257.25" velocity="3.8397"/>
+        <limit lower="${radians(-175)}" upper="${radians(240)}" effort="257.25" velocity="${radians(220)}"/>
     </joint>
     <joint name="${prefix}joint_4_r" type="revolute">
@@ -124,5 +124,5 @@
         <origin xyz="0.640 0 0.200" rpy="0 0 0" />
         <axis xyz="-1 0 0" />
-        <limit lower="-3.1415" upper="3.1415" effort="74.97" velocity="7.1558"/>
+        <limit lower="${radians(-180)}" upper="${radians(-180)}" effort="74.97" velocity="${radians(410)}"/>
     </joint>
     <joint name="${prefix}joint_5_b" type="revolute">
@@ -131,5 +131,5 @@
         <origin xyz="0 0 0" rpy="0 0 0" />
         <axis xyz="0 -1 0" />
-        <limit lower="-2.3562" upper="2.3562" effort="44.69" velocity="7.1558"/>
+        <limit lower="${radians(-135)}" upper="${radians(135)}" effort="44.69" velocity="${radians(410)}"/>
     </joint>
     <joint name="${prefix}joint_6_t" type="revolute">
@@ -138,5 +138,5 @@
         <origin xyz="0 0 0" rpy="0 0 0" />
         <axis xyz="-1 0 0" />
-        <limit lower="-6.2832" upper="6.2832" effort="14.80" velocity="10.6465"/>
+        <limit lower="${radians(-360)}" upper="${radians(360)}" effort="14.80" velocity="${radians(610)}"/>
     </joint>
     <joint name="${prefix}joint_6_t-tool0" type="fixed">
