Commit message: es_support: use xacro.load_yaml(..) instead (#637)
Plain `load_yaml(..)` is deprecated.

File: motoman_es_support/urdf/es165_macro.xacro (robot description, xacro)
@@ -163,5 +163,5 @@
     <!-- end of link list -->
     <!-- joint list -->
-    <xacro:property name="velocities" value="${load_yaml(joint_velocities_file)}" />
+    <xacro:property name="velocities" value="${xacro.load_yaml(joint_velocities_file)}" />
     <joint name="${prefix}joint_1_s" type="revolute">
       <origin xyz="0 0 0.450" rpy="0 0 0"/>

File: motoman_es_support/urdf/es200_120_macro.xacro (robot description, xacro)
@@ -161,5 +161,5 @@
     <!-- end of link list -->
     <!-- joint list -->
-    <xacro:property name="velocities" value="${load_yaml(joint_velocities_file)}" />
+    <xacro:property name="velocities" value="${xacro.load_yaml(joint_velocities_file)}" />
     <joint name="${prefix}joint_1_s" type="revolute">
       <origin xyz="0 0 0.450" rpy="0 0 0"/>
